File: BenEater-6502.kicad_pcb (KiCad board)
At the start: 2 copper layers, 157.5 x 180.3 mm, 93 parts, among them J1 Serial Header, J2 Arduino Mega, J3 Expansion, J4 Logic Probe, J5 Barrel Jack, SW1 Step, SW11 NMI, SW12 RESET, SW2 Run / Step, SW3 Clk Source, SW5 Power, U1 LM555, U10 74LS00, U11 W65C22NxP, U12 HM62256BLP, U13 W65C51NxP, U14 MAX232N, U15 LM555, U2 LM555, U3 LM555, U4 74LS04, U5 74LS08, U6 74LS32, U7 W65C02SxP, U8 28C256, U9 LCD-16X2, X1 ACO-xxxMHz, Y1 Crystal

Commit message: intermediate commit
Parts:
- removed Buttom1: Buttom, Button_Switch_THT:SW_PUSH_6mm_H5mm
- removed D10: A10-A15/CLK/IRQ, digikey-footprints:LED_Bar_Graph_LTA-1000
- removed D9: A0-A9, digikey-footprints:LED_Bar_Graph_LTA-1000
- removed RN1: D0-7, Resistor_THT:R_Array_SIP11
- removed RN2: A0-A9, Resistor_THT:R_Array_SIP11
- removed RN3: A10-A15/CLK/IRQ, Resistor_THT:R_Array_SIP11
- removed SW11: NMI, Button_Switch_THT:SW_PUSH_6mm_H5mm
- removed SW12: RESET, Button_Switch_THT:SW_PUSH_6mm_H5mm
- added Bottom1: Bottom, Button_Switch_THT:SW_PUSH_6mm_H5mm, F.Cu at (-46.9, 78.8)
- added C23: 1uf, Capacitor_THT:C_Disc_D4.3mm_W1.9mm_P5.00mm, F.Cu at (-126.7, 146.4)
- added C24: 1uf, Capacitor_THT:C_Disc_D4.3mm_W1.9mm_P5.00mm, F.Cu at (-126.7, 149.9)
- added C25: .1uf, Capacitor_THT:C_Disc_D4.3mm_W1.9mm_P5.00mm, F.Cu at (-126.7, 153.3)
- added C26: .1uf, Capacitor_THT:C_Disc_D4.3mm_W1.9mm_P5.00mm, F.Cu at (-126.7, 156.8)
- added D6: Power, LED_THT:LED_D5.0mm, F.Cu at (30.5, 20.3)
- added J10: Conn_01x03_Pin, Connector_PinSocket_1.27mm:PinSocket_1x03_P1.27mm_Vertical, F.Cu at (-117.8, 136.0)
- added J6: Conn_02x20_Counter_Clockwise, Connector_PinSocket_1.27mm:PinSocket_2x20_P1.27mm_Vertical, F.Cu at (-19.3, 78.5)
- added J7: Conn_01x09, Connector_PinSocket_1.27mm:PinSocket_1x09_P1.27mm_Vertical, F.Cu at (-136.7, 115.9)
- added J8: Conn_01x09, Connector_PinSocket_1.27mm:PinSocket_1x09_P1.27mm_Vertical, F.Cu at (-132.1, 115.9)
- added J9: Conn_01x09, Connector_PinSocket_1.27mm:PinSocket_1x09_P1.27mm_Vertical, F.Cu at (-127.5, 115.9)
- added R24: 1M, Resistor_THT:R_Axial_DIN0207_L6.3mm_D2.5mm_P7.62mm_Horizontal, F.Cu at (-124.5, 129.7)
- added SW4: RESET, Button_Switch_THT:SW_PUSH_6mm_H5mm, F.Cu at (-46.3, 62.2)
- added SW6: Power, digikey-footprints:Switch_Slide_11.6x4mm_EG1218, F.Cu at (31.8, 29.2)
- added U16: MAX232N, digikey-footprints:DIP-16_W7.62mm, F.Cu at (-137.4, 137.1)
- C1, C3: value 0.1µF -> 0.01µF
- C10, C11, C12, C13, C14, C9: value .1uf -> 0.1µF
- C16, C17, C18, C19: value 1uf -> .1uf
- C2: value 0.01µF -> 1µF; footprint Capacitor_THT:C_Disc_D4.3mm_W1.9mm_P5.00mm -> Capacitor_THT:CP_Radial_D5.0mm_P2.00mm
- C20: value 20pf -> 1uf
- C21: value .1uf -> 1uf
- C22: value 220nF -> 20pf
- C5: value 0.01µF -> 0.1µF
- C6: value 1µF -> 0.01µF; footprint Capacitor_THT:CP_Radial_D5.0mm_P2.00mm -> Capacitor_THT:C_Disc_D4.3mm_W1.9mm_P5.00mm
- C7: value 0.01µF -> 220nF
- D8: value DATA -> SB140; footprint digikey-footprints:LED_Bar_Graph_LTA-1000 -> Diode_THT:D_DO-41_SOD81_P10.16mm_Horizontal
- J1: value Serial Header -> Conn_01x03_Pin; footprint Connector_PinHeader_2.54mm:PinHeader_1x03_P2.54mm_Vertical -> Connector_PinSocket_1.27mm:PinSocket_1x03_P1.27mm_Vertical
- J2: value Arduino Mega -> Conn_01x02; footprint Connector_PinSocket_2.54mm:PinSocket_2x16_P2.54mm_Vertical -> Connector_PinSocket_1.27mm:PinSocket_1x02_P1.27mm_Vertical
- J3: value Expansion -> Barrel Jack; footprint Connector_PinSocket_2.54mm:PinSocket_2x16_P2.54mm_Vertical -> Connector_BarrelJack:BarrelJack_Horizontal
- J5: value Barrel Jack -> Conn_02x20_Counter_Clockwise; footprint Connector_BarrelJack:BarrelJack_Horizontal -> Connector_PinSocket_1.27mm:PinSocket_2x20_P1.27mm_Vertical
- R10, R14: value 220 -> 1k
- R11, R17, R18, R3, R6: value 1K -> 220
- R12: value 1K -> 1k
- R13: value 1M -> 47k
- R15: value 1K -> 10K
- R20: value 10K -> 1K
- R21: value 47k -> 1K
- R22, R23: value 1k -> 1K
- R4: value 1M -> 1K
- R5: value 1K -> 1M
- R7, R8: value 220 -> 1K
- SW5: value Power -> NMI; footprint digikey-footprints:Switch_Slide_11.6x4mm_EG1218 -> Button_Switch_THT:SW_PUSH_6mm_H5mm
- U10: value 74LS00 -> HM62256BLP; footprint Package_DIP:DIP-14_W7.62mm -> Package_DIP:DIP-28_W15.24mm
- U12: value HM62256BLP -> LCD-16X2; footprint Package_DIP:DIP-28_W15.24mm -> 8bit-custom-footprints:MODULE_LCD-16X2
- U13: value W65C51NxP -> 74LS00; footprint Package_DIP:DIP-28_W15.24mm -> Package_DIP:DIP-14_W7.62mm
- U14: value MAX232N -> W65C22NxP; footprint digikey-footprints:DIP-16_W7.62mm -> Package_DIP:DIP-40_W15.24mm
- U15: value LM555 -> W65C51NxP; footprint Package_DIP:DIP-8_W7.62mm -> Package_DIP:DIP-28_W15.24mm
- U7: value W65C02SxP -> LM555; footprint Package_DIP:DIP-40_W15.24mm -> Package_DIP:DIP-8_W7.62mm
- U8: value 28C256 -> W65C02SxP; footprint Package_DIP:DIP-28_W15.24mm -> Package_DIP:DIP-40_W15.24mm
- U9: value LCD-16X2 -> 28C256; footprint 8bit-custom-footprints:MODULE_LCD-16X2 -> Package_DIP:DIP-28_W15.24mm
- moved Y1 298.5 mm to (-135.0, 131.0)
- moved C20 288.9 mm to (-126.7, 136.1)
- moved C21 258.1 mm to (-126.7, 139.5)
- moved U9 251.9 mm to (-119.0, 77.1)
- moved D8 250.3 mm to (-155.6, 153.5), turned to 0 degrees
- moved U8 249.9 mm to (-155.8, 57.7)
- moved C16 248.2 mm to (-82.2, 84.5)
- moved C17 247.8 mm to (-82.2, 87.9)
- moved C18 247.4 mm to (-82.2, 91.4)
- moved RV2 240.2 mm to (-72.5, 82.3), turned to 0 degrees
- moved D5 238.0 mm to (-82.0, 77.2), turned to 0 degrees
- moved U12 233.2 mm to (-116.0, 36.9)
- moved U13 226.3 mm to (-86.5, 57.7)
- moved C19 222.1 mm to (-47.3, 121.3)
- moved U10 219.9 mm to (-100.7, 77.1)
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Connections:
- C1 pad 1: VCC -> Net-(U1-CV)
- C1 pad 2: GND -> Earth
- C16 pad 1: Net-(U14-C2+) -> +5V
- C16 pad 2: Net-(U14-C2-) -> Earth
- C17 pad 1: Net-(U14-C1+) -> +5V
- C17 pad 2: Net-(U14-C1-) -> Earth
- C18 pad 1: Net-(U14-VS+) -> +5V
- C19 pad 1: Net-(U14-VS-) -> +5V
- C2 pad 1: Net-(U2-CV) -> Net-(U1-THR)
- C2 pad 2: GND -> Earth
- C20 pad 1: Net-(U13-XTAL1) -> Net-(U16-C1-)
- C20 pad 2: Earth -> Net-(U16-C1+)
- C21 pad 1: +5V -> Net-(U16-C2-)
- C21 pad 2: Earth -> Net-(U16-C2+)
- C22 pad 1: Net-(U15-THR) -> Net-(U15-XTAL2)
- C22 pad 2: GND -> Earth
- C3 pad 1: Net-(U2-DIS) -> Net-(U2-TR)
- C3 pad 2: GND -> Earth
- C4 pad 1: Net-(U3-CV) -> Net-(U2-CV)
- C4 pad 2: GND -> Earth
- C5 pad 1: Net-(U1-CV) -> Net-(U2-DIS)
- C5 pad 2: GND -> Earth
- C6 pad 1: Net-(U1-THR) -> Net-(U3-CV)
- C6 pad 2: GND -> Earth
- C7 pad 1: Net-(U2-TR) -> Net-(U7-THR)
- C7 pad 2: GND -> Earth
- C8 pad 1: VCC -> +5V
- C8 pad 2: GND -> Earth
- C9 pad 1: /Reset -> +5V
- D5 pad 2: /Reset -> /IRQ
- D8 pad 1: /D0 -> Net-(D8-K)
- D8 pad 2: /D1 -> /IRQ
- J1 pad 1: Earth -> Net-(J1-Pin_1)
- J1 pad 2: Net-(J1-Pin_2) -> /Reset
- J2 pad 1: /A0 -> Net-(J2-Pin_1)
- J2 pad 2: /D0 -> Earth
- J3 pad 1: /A0 -> Net-(J2-Pin_1)
- J3 pad 2: /D0 -> Earth
- J3 pad 3: /A1 -> (no net)
- J5 pad 1: Earth -> /A0
- J5 pad 2: Net-(SW5-B) -> /A1
- J5 pad 3: (no net) -> /A2
- Left1 pad 2: Net-(U11-PA3) -> Net-(U14-PA1)
- Middle1 pad 2: Net-(U11-PA0) -> Net-(U14-PA2)
- R1 pad 1: VCC -> +5V
- R10 pad 1: GND -> +5V
- R10 pad 2: Net-(D3-K) -> /HLT
- R11 pad 1: +5V -> Net-(D4-K)
- R11 pad 2: /Reset -> Earth
- R12 pad 1: +5V -> Net-(U7-THR)
- R12 pad 2: Net-(U7-RDY) -> Net-(R12-Pad2)
- R13 pad 1: Net-(U13-XTAL2) -> Net-(R12-Pad2)
- R13 pad 2: Net-(U13-XTAL1) -> Earth
- R14 pad 1: Net-(J4-Pin_1) -> +5V
- R14 pad 2: Net-(D11-A) -> Net-(J1-Pin_1)
- R15 pad 1: Net-(U11-PA0) -> Net-(U8-~{NMI})
- R16 pad 1: Net-(U11-PA1) -> +5V
- R16 pad 2: +5V -> Net-(U8-RDY)
- R17 pad 1: Net-(U11-PA2) -> +5V
- R17 pad 2: +5V -> Net-(D6-A)
- R18 pad 1: Net-(U11-PA3) -> Net-(J4-Pin_1)
- R18 pad 2: +5V -> Net-(D11-A)
- R19 pad 1: Net-(U11-PA4) -> Net-(U14-PA0)
- R20 pad 1: Net-(U7-~{NMI}) -> Net-(U14-PA1)
- R21 pad 1: Net-(R21-Pad1) -> Net-(U14-PA2)
- R21 pad 2: GND -> +5V
- R22 pad 1: Net-(U15-THR) -> Net-(U14-PA3)
- R22 pad 2: Net-(R21-Pad1) -> +5V
- R23 pad 1: VCC -> Net-(U14-PA4)
- R23 pad 2: /Reset -> +5V
- R3 pad 1: VCC -> Earth
- R3 pad 2: Net-(U2-TR) -> Net-(D1-K)
- R4 pad 1: VCC -> +5V
- R4 pad 2: Net-(U2-DIS) -> Net-(U2-TR)
- R5 pad 1: VCC -> +5V
- R5 pad 2: Net-(SW2-A) -> Net-(U2-DIS)
- R6 pad 1: VCC -> Earth
- R6 pad 2: Net-(SW2-C) -> Net-(D2-K)
- R7 pad 1: Net-(D4-K) -> +5V
- R7 pad 2: GND -> Net-(SW2-A)
- R8 pad 1: GND -> +5V
- R8 pad 2: Net-(D1-K) -> Net-(SW2-C)
- R9 pad 1: GND -> Earth
- R9 pad 2: Net-(D2-K) -> Net-(D3-K)
- RV2 pad 2: Net-(U9-VO) -> Net-(U12-VO)
- RV2 pad 3: Earth -> unconnected-(RV2-Pad3)
- Right1 pad 2: Net-(U11-PA4) -> Net-(U14-PA3)
- SW1 pad 1: GND -> Earth
- SW2 pad 2: GND -> Earth
- SW5 pad 1: unconnected-(SW5-A-Pad1) -> Earth
- SW5 pad 2: Net-(SW5-B) -> Net-(U8-~{NMI})
- Top1 pad 2: Net-(U11-PA1) -> Net-(U14-PA0)
- U1 pad 1: GND -> Earth
- U1 pad 4: VCC -> +5V
- U1 pad 8: VCC -> +5V
- U10 pad 1: /A15 -> /A14
- U10 pad 10: Net-(U10-1Y) -> /A0
- U10 pad 11: Net-(U10-4Y) -> /D0
- U10 pad 12: /R/W -> /D1
- U10 pad 13: /R/W -> /D2
- U10 pad 14: +5V -> Earth
- U10 pad 2: /A15 -> /A12
- U10 pad 3: Net-(U10-1Y) -> /A7
- U10 pad 4: /CLK -> /A6
- U10 pad 5: Net-(U10-1Y) -> /A5
- U10 pad 6: Net-(U10-2Y) -> /A4
- U10 pad 7: Earth -> /A3
- U10 pad 8: Net-(U10-3Y) -> /A2
- U10 pad 9: unconnected-(U10-3B-Pad9) -> /A1
- U11 pad 17: /HLT -> unconnected-(U11-PB7-Pad17)
- U11 pad 2: Net-(U11-PA0) -> /RTSVia
- U11 pad 21: Net-(D7-K) -> Net-(D5-K)
- U11 pad 23: Net-(U10-3Y) -> Net-(U11-~{CS2})
- U11 pad 3: Net-(U11-PA1) -> unconnected-(U11-PA1-Pad3)
- U11 pad 4: Net-(U11-PA2) -> unconnected-(U11-PA2-Pad4)
- U11 pad 5: Net-(U11-PA3) -> unconnected-(U11-PA3-Pad5)
- U11 pad 6: Net-(U11-PA4) -> unconnected-(U11-PA4-Pad6)
- U12 pad 1: /A14 -> Earth
- U12 pad 10: /A0 -> unconnected-(U12-DB3-Pad10)
- U12 pad 11: /D0 -> Net-(U11-PB0)
- U12 pad 12: /D1 -> Net-(U11-PB1)
- U12 pad 13: /D2 -> Net-(U11-PB2)
- U12 pad 14: Earth -> Net-(U11-PB3)
- U12 pad 15: /D3 -> +5V
- U12 pad 16: /D4 -> Earth
- U12 pad 2: /A12 -> +5V
- U12 pad 3: /A7 -> Net-(U12-VO)
- U12 pad 4: /A6 -> Net-(U11-PB4)
- U12 pad 5: /A5 -> Net-(U11-PB5)
- U12 pad 6: /A4 -> Net-(U11-PB6)
- U12 pad 7: /A3 -> unconnected-(U12-DB0-Pad7)
- U12 pad 8: /A2 -> unconnected-(U12-DB1-Pad8)
- U12 pad 9: /A1 -> unconnected-(U12-DB2-Pad9)
- U13 pad 1: Earth -> /A15
- U13 pad 10: /TxD -> /A14
- U13 pad 11: unconnected-(U13-~{DTR}-Pad11) -> (no net)
- U13 pad 12: /RxD -> (no net)
- U13 pad 13: /A0 -> (no net)
- U13 pad 14: /A1 -> (no net)
- U13 pad 2: /A12 -> /A15
- U13 pad 3: Net-(U10-3Y) -> Net-(U9-~{CS})
- U13 pad 4: /IRQ -> Net-(U9-~{CS})
- U13 pad 5: unconnected-(U13-RxC-Pad5) -> /CLK
- U13 pad 6: Net-(U13-XTAL1) -> Net-(U10-~{CS})
- U13 pad 7: Net-(U13-XTAL2) -> (no net)
- U13 pad 8: unconnected-(U13-~{RTS}-Pad8) -> /CS2
- U13 pad 9: unconnected-(U13-~{CTS}-Pad9) -> Net-(U9-~{CS})
- U14 pad 1: Net-(U14-C1+) -> Earth
- U14 pad 11: /TxD -> unconnected-(U14-PB1-Pad11)
- U14 pad 12: /RxD -> unconnected-(U14-PB2-Pad12)
- U14 pad 13: Net-(J1-Pin_2) -> unconnected-(U14-PB3-Pad13)
- U14 pad 14: Net-(J1-Pin_3) -> unconnected-(U14-PB4-Pad14)
- U14 pad 15: Earth -> unconnected-(U14-PB5-Pad15)
- U14 pad 16: +5V -> unconnected-(U14-PB6-Pad16)
- U14 pad 2: Net-(U14-VS+) -> Net-(U14-PA0)
- U14 pad 3: Net-(U14-C1-) -> Net-(U14-PA1)
- U14 pad 4: Net-(U14-C2+) -> Net-(U14-PA2)
- U14 pad 5: Net-(U14-C2-) -> Net-(U14-PA3)
- U14 pad 6: Net-(U14-VS-) -> Net-(U14-PA4)
- U15 pad 1: GND -> Earth
- U15 pad 2: Net-(U15-THR) -> /A12
- U15 pad 3: unconnected-(U15-Q-Pad3) -> /CS2
- U15 pad 4: VCC -> /Reset
- U15 pad 6: Net-(U15-THR) -> Net-(U15-XTAL1)
- U15 pad 7: /Reset -> Net-(U15-XTAL2)
- U15 pad 8: VCC -> Net-(J10-Pin_1)
- U2 pad 1: GND -> Earth
- U2 pad 4: VCC -> +5V
- U2 pad 8: VCC -> +5V
- U3 pad 1: GND -> Earth
- U3 pad 6: GND -> Earth
- U3 pad 8: VCC -> +5V
- U4 pad 10: (no net) -> /CS2Via2
- U4 pad 11: (no net) -> Net-(U11-~{CS2})
- U4 pad 12: /Clock/~{CLK} -> Net-(U9-~{OE})
- U4 pad 13: Net-(D4-A) -> /R/W
- U4 pad 3: (no net) -> Net-(R12-Pad2)
- U4 pad 4: (no net) -> Net-(J1-Pin_3)
- U4 pad 5: (no net) -> /HLT
- U4 pad 6: (no net) -> Net-(U4-Pad6)
- U4 pad 8: Net-(U4-Pad8) -> /Clock/~{CLK}
- U4 pad 9: /HLT -> Net-(D4-A)
- U5 pad 10: Net-(U4-Pad8) -> Net-(U4-Pad6)
- U5 pad 11: Net-(U12-~{OE}) -> Net-(U10-~{OE})
- U6 pad 4: (no net) -> /A4
- U6 pad 5: (no net) -> /CS2
- U6 pad 6: (no net) -> Net-(U11-~{CS2})
- U7 pad 1: unconnected-(U7-~{VP}-Pad1) -> Earth
- U7 pad 2: Net-(U7-RDY) -> Net-(U7-THR)
- U7 pad 4: /IRQ -> +5V
- U7 pad 6: Net-(U7-~{NMI}) -> Net-(U7-THR)
- U7 pad 7: /Sync -> Net-(J1-Pin_1)
- U8 pad 1: /A14 -> unconnected-(U8-~{VP}-Pad1)
- U8 pad 10: /A0 -> /A1
- U8 pad 11: /D0 -> /A2
- U8 pad 12: /D1 -> /A3
- U8 pad 13: /D2 -> /A4
- U8 pad 14: Earth -> /A5
- U8 pad 15: /D3 -> /A6
- U8 pad 16: /D4 -> /A7
- U8 pad 17: /D5 -> /A8
- U8 pad 18: /D6 -> /A9
- U8 pad 19: /D7 -> /A10
- U8 pad 2: /A12 -> Net-(U8-RDY)
- U8 pad 20: Net-(U10-1Y) -> /A11
- U8 pad 21: /A10 -> Earth
- U8 pad 22: Net-(U10-4Y) -> /A12
- U8 pad 23: /A11 -> /A13
- U8 pad 24: /A9 -> /A14
- U8 pad 25: /A8 -> /A15
- U8 pad 26: /A13 -> /D7
- U8 pad 27: +5V -> /D6
- U8 pad 28: +5V -> /D5
- U8 pad 3: /A7 -> unconnected-(U8-ϕ1-Pad3)
- U8 pad 4: /A6 -> /IRQ
- U8 pad 5: /A5 -> unconnected-(U8-~{ML}-Pad5)
- U8 pad 6: /A4 -> Net-(U8-~{NMI})
- U8 pad 7: /A3 -> /Sync
- U8 pad 8: /A2 -> +5V
- U8 pad 9: /A1 -> /A0
- U9 pad 1: Earth -> /A14
- U9 pad 10: unconnected-(U9-DB3-Pad10) -> /A0
- U9 pad 11: Net-(U11-PB0) -> /D0
- U9 pad 12: Net-(U11-PB1) -> /D1
- U9 pad 13: Net-(U11-PB2) -> /D2
- U9 pad 14: Net-(U11-PB3) -> Earth
- U9 pad 15: +5V -> /D3
- U9 pad 16: Earth -> /D4
- U9 pad 2: +5V -> /A12
- U9 pad 3: Net-(U9-VO) -> /A7
- U9 pad 4: Net-(U11-PB4) -> /A6
- U9 pad 5: Net-(U11-PB5) -> /A5
- U9 pad 6: Net-(U11-PB6) -> /A4
- U9 pad 7: unconnected-(U9-DB0-Pad7) -> /A3
- U9 pad 8: unconnected-(U9-DB1-Pad8) -> /A2
- U9 pad 9: unconnected-(U9-DB2-Pad9) -> /A1
- X1 pad 7: GND -> Earth
- Y1 pad 1: Net-(U13-XTAL2) -> Net-(U15-XTAL2)
- Y1 pad 2: Net-(U13-XTAL1) -> Net-(U15-XTAL1)
Routing:
- net Earth: track 720.5 -> 0.00 mm
- net +5V: track 498.0 -> 0.00 mm
- net /CLK: track 463.4 -> 0.00 mm, vias 2 -> 0
- net /R/W: track 386.4 -> 0.00 mm
- net /Reset: track 378.6 -> 0.00 mm
- net /IRQ: track 360.7 -> 0.00 mm, vias 2 -> 0
- net /D6: track 353.3 -> 0.00 mm, vias 2 -> 0
- net /D7: track 348.9 -> 0.00 mm, vias 1 -> 0
- net /D3: track 348.6 -> 0.00 mm, vias 2 -> 0
- net /D4: track 342.9 -> 0.00 mm, vias 1 -> 0
- net /A1: track 341.2 -> 0.00 mm, vias 4 -> 0
- net /A2: track 333.6 -> 0.00 mm, vias 4 -> 0
- net /A4: track 332.3 -> 0.00 mm, vias 1 -> 0
- net /A9: track 331.8 -> 0.00 mm, vias 2 -> 0
- net /D5: track 322.9 -> 0.00 mm, vias 1 -> 0
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Other:
- outline, holes or cut-outs redrawn
- board text added: "Clock Generator"
- board text added: "Clock Run/Step"
- board text added: "Clock Step"
- board text added: "Power Input"

Commit message: interm commit
Parts:
- added C27: .1uf, Capacitor_THT:C_Disc_D4.3mm_W1.9mm_P5.00mm, F.Cu at (60.9, 73.9)
- added D10: 1N4001, Diode_THT:D_DO-41_SOD81_P10.16mm_Horizontal, F.Cu at (21.6, 41.3)
- added D9: 1N4001, Diode_THT:D_DO-41_SOD81_P10.16mm_Horizontal, F.Cu at (38.1, 31.7)
- added J11: Halt, Connector_Pin:Pin_D1.0mm_L10.0mm, F.Cu at (17.8, 48.2)
- added J12: Conn_01x10, Connector_PinSocket_1.27mm:PinSocket_1x10_P1.27mm_Vertical, F.Cu at (67.7, 159.4)
- added J13: Conn_01x10, Connector_PinSocket_1.27mm:PinSocket_1x10_P1.27mm_Vertical, F.Cu at (43.5, 159.5)
- added J14: Conn_01x10, Connector_PinSocket_1.27mm:PinSocket_1x10_P1.27mm_Vertical, F.Cu at (20.7, 130.7)
- added R25: 1K, Resistor_THT:R_Axial_DIN0207_L6.3mm_D2.5mm_P7.62mm_Horizontal, F.Cu at (89.5, 48.0)
- moved C26 295.7 mm to (168.9, 160.6), turned to -90 degrees
- moved J8 288.6 mm to (149.5, 178.9), turned to 90 degrees
- moved J9 285.6 mm to (149.5, 185.5), turned to 90 degrees
- moved U16 283.6 mm to (144.6, 167.0), turned to 90 degrees
- moved C23 283.0 mm to (154.9, 174.6)
- moved C21 281.2 mm to (152.3, 174.6), turned to 180 degrees
- moved C20 274.1 mm to (144.7, 174.6), turned to 180 degrees
- moved C24 268.0 mm to (139.8, 178.9)
- moved J7 266.7 mm to (122.0, 180.8), turned to 90 degrees
- moved U12 263.7 mm to (130.3, 131.0)
- moved C25 256.7 mm to (129.8, 164.4), turned to -90 degrees
- moved U15 254.1 mm to (91.5, 174.6), turned to 90 degrees
- moved D8 253.4 mm to (96.4, 180.9), turned to 180 degrees
- moved Y1 248.1 mm to (108.0, 180.9), turned to 180 degrees
- moved C22 241.2 mm to (109.3, 192.4), turned to 180 degrees
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Connections:
- J2 pad 1: Net-(J2-Pin_1) -> Net-(D9-A)
- J2 pad 2: Earth -> Net-(D10-K)
- J3 pad 1: Net-(J2-Pin_1) -> Net-(D9-A)
- J3 pad 2: Earth -> Net-(D10-K)
- R10 pad 2: /HLT -> /Clock/Halt
- SW6 pad 2: Net-(J2-Pin_1) -> Net-(D9-K)
- U11 pad 14: Net-(U11-PB4) -> Net-(U11-PB3)
- U11 pad 23: Net-(U11-~{CS2}) -> /CS2
- U11 pad 3: unconnected-(U11-PA1-Pad3) -> Net-(J14-Pin_3)
- U11 pad 4: unconnected-(U11-PA2-Pad4) -> Net-(J14-Pin_4)
- U11 pad 5: unconnected-(U11-PA3-Pad5) -> Net-(J14-Pin_5)
- U11 pad 6: unconnected-(U11-PA4-Pad6) -> Net-(J14-Pin_6)
- U11 pad 7: unconnected-(U11-PA5-Pad7) -> Net-(J14-Pin_7)
- U11 pad 8: unconnected-(U11-PA6-Pad8) -> Net-(J14-Pin_8)
- U11 pad 9: unconnected-(U11-PA7-Pad9) -> Net-(J14-Pin_9)
- U12 pad 4: Net-(U11-PB4) -> Net-(U11-PB3)
- U13 pad 11: (no net) -> Net-(U10-~{CS})
- U13 pad 12: (no net) -> Net-(U13-Pad12)
- U13 pad 13: (no net) -> /CS2
- U13 pad 6: Net-(U10-~{CS}) -> Net-(U13-Pad12)
- U14 pad 10: unconnected-(U14-PB0-Pad10) -> Net-(J12-Pin_2)
- U14 pad 11: unconnected-(U14-PB1-Pad11) -> Net-(J12-Pin_3)
- U14 pad 12: unconnected-(U14-PB2-Pad12) -> Net-(J12-Pin_4)
- U14 pad 13: unconnected-(U14-PB3-Pad13) -> Net-(J12-Pin_5)
- U14 pad 14: unconnected-(U14-PB4-Pad14) -> Net-(J12-Pin_6)
- U14 pad 15: unconnected-(U14-PB5-Pad15) -> Net-(J12-Pin_7)
- U14 pad 16: unconnected-(U14-PB6-Pad16) -> Net-(J12-Pin_8)
- U14 pad 17: unconnected-(U14-PB7-Pad17) -> Net-(J12-Pin_9)
- U14 pad 7: unconnected-(U14-PA5-Pad7) -> Net-(J13-Pin_7)
- U14 pad 8: unconnected-(U14-PA6-Pad8) -> Net-(J13-Pin_8)
- U14 pad 9: unconnected-(U14-PA7-Pad9) -> Net-(J13-Pin_9)
- U4 pad 11: Net-(U11-~{CS2}) -> /A4
- U4 pad 5: /HLT -> /Clock/Halt
- U6 pad 4: /A4 -> (no net)
- U6 pad 5: /CS2 -> (no net)
- U6 pad 6: Net-(U11-~{CS2}) -> (no net)
Other:
- board text added: "CPU"
- board text added: "Control Logic"
- board text added: "Display"
- board text added: "Expainsion/Mega"
- board text added: "Expansion Via"
- board text added: "Logic Probe"
- board text added: "Navagation"
- board text added: "RAM"
- board text added: "ROM"
- board text added: "Reset & NMI"
- board text added: "Serial"

Commit message: An other interm relase
Parts:
- added C28: .1uf, Capacitor_THT:C_Disc_D4.3mm_W1.9mm_P5.00mm, F.Cu at (60.9, 103.6)
- added U17: 74LS08, Package_DIP:DIP-14_W7.62mm, F.Cu at (59.8, 81.8)
- J11: value Halt -> HLT
- J12, J13, J14: footprint Connector_PinSocket_1.27mm:PinSocket_1x10_P1.27mm_Vertical -> Connector_PinSocket_2.54mm:PinSocket_1x10_P2.54mm_Vertical
- J5, J6: footprint Connector_PinSocket_1.27mm:PinSocket_2x20_P1.27mm_Vertical -> Connector_PinSocket_2.54mm:PinSocket_2x20_P2.54mm_Vertical
- J7, J8, J9: footprint Connector_PinSocket_1.27mm:PinSocket_1x09_P1.27mm_Vertical -> Connector_PinSocket_2.54mm:PinSocket_1x09_P2.54mm_Vertical
- moved J5 15.4 mm to (52.9, 169.0)
Connections:
- net Net-(U10-~{OE}) renamed /RAMOE
- J11 pad 1: /Clock/Halt -> /HLT
- R10 pad 2: /Clock/Halt -> /HLT
- U10 pad 20: Net-(U10-~{CS}) -> /RAMCS
- U11 pad 14: Net-(U11-PB3) -> Net-(U11-PB4)
- U12 pad 4: Net-(U11-PB3) -> Net-(U11-PB4)
- U13 pad 1: /A15 -> /Control Logic/A15
- U13 pad 10: /A14 -> /CS2Via2
- U13 pad 11: Net-(U10-~{CS}) -> (no net)
- U13 pad 12: Net-(U13-Pad12) -> (no net)
- U13 pad 13: /CS2 -> (no net)
- U13 pad 2: /A15 -> /Control Logic/A15
- U13 pad 3: Net-(U9-~{CS}) -> /ROMCS
- U13 pad 4: Net-(U9-~{CS}) -> /ROMCS
- U13 pad 5: /CLK -> /Control Logic/CLK
- U13 pad 6: Net-(U13-Pad12) -> /RAMCS
- U13 pad 9: Net-(U9-~{CS}) -> Net-(U13-Pad9)
- U4 pad 11: /A4 -> Net-(U17-Pad8)
- U4 pad 14: VCC -> +5V
- U4 pad 5: /Clock/Halt -> /HLT
- U4 pad 7: GND -> Earth
- U5 pad 12: /A13 -> /Control Logic/A13
- U5 pad 13: /A14 -> /Control Logic/A12
- U5 pad 14: VCC -> +5V
- U5 pad 7: GND -> Earth
- U6 pad 14: VCC -> +5V
- U6 pad 7: GND -> Earth
- U9 pad 20: Net-(U9-~{CS}) -> /ROMCS
- X1 pad 14: VCC -> +5V

Commit message: Getting closer
Parts:
- moved D8 69.2 mm to (160.2, 154.2), turned to 0 degrees
- moved C26 49.3 mm to (129.4, 190.1), turned to 0 degrees
- moved Y1 37.7 mm to (134.4, 154.1)
- moved J9 30.6 mm to (169.8, 162.5), turned to 0 degrees
- moved C22 30.5 mm to (134.4, 175.1), turned to -90 degrees
- moved R24 30.5 mm to (134.4, 169.9), turned to 90 degrees
- moved J10 28.2 mm to (106.8, 154.1), turned to 90 degrees
- moved C24 27.1 mm to (150.9, 154.2)
- moved U15 21.9 mm to (106.8, 159.0), turned to 0 degrees
- moved C23 20.6 mm to (141.7, 190.3)
- moved C20 20.3 mm to (146.7, 154.3)
- moved J7 19.8 mm to (129.3, 162.4), turned to 0 degrees
- moved J8 17.9 mm to (156.7, 162.5), turned to 0 degrees
- moved J14 17.8 mm to (37.9, 135.7)
- moved C25 12.9 mm to (122.0, 154.1), turned to 180 degrees
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Other:
- board text added: "BE6502 V2 Rev A"

Commit message: Fix Oops...
Parts:
- removed D10: 1N4001, Diode_THT:D_DO-41_SOD81_P10.16mm_Horizontal
- removed U8: W65C02SxP, Package_DIP:DIP-40_W15.24mm
- C15, C16, C17, C18, C19, C25, C26, C27, C28: value .1uf -> 0.1uf
- J1, J10: footprint Connector_PinSocket_1.27mm:PinSocket_1x03_P1.27mm_Vertical -> Connector_PinSocket_2.54mm:PinSocket_1x03_P2.54mm_Vertical
- J2: footprint Connector_PinSocket_1.27mm:PinSocket_1x02_P1.27mm_Vertical -> Connector_PinSocket_2.54mm:PinSocket_1x02_P2.54mm_Vertical
- moved D7 54.9 mm to (87.1, 152.0)
- moved R19 54.9 mm to (81.3, 143.2)
- moved R20 54.9 mm to (81.3, 148.1)
- moved R21 54.9 mm to (81.4, 152.9)
- moved R22 54.9 mm to (81.4, 157.7)
- moved C19 54.9 mm to (87.1, 142.4)
- moved R23 54.9 mm to (81.5, 162.2)
- moved C18 51.0 mm to (83.1, 120.3)
- moved D5 51.0 mm to (83.1, 115.5)
- moved J14 19.0 mm to (18.9, 135.7)
- moved U11 19.0 mm to (18.9, 130.6)
- moved J13 18.9 mm to (18.9, 162.6)
- moved U14 18.9 mm to (18.9, 158.1)
- moved J12 18.9 mm to (47.6, 162.6)
- moved C27 5.01 mm to (65.9, 73.9), turned to 180 degrees
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Connections:
- J2 pad 2: Net-(D10-K) -> Earth
- J3 pad 2: Net-(D10-K) -> Earth
- U13 pad 1: /Control Logic/A15 -> /A15
- U13 pad 11: (no net) -> /CS2Via2
- U13 pad 12: (no net) -> /ROMCS
- U13 pad 13: (no net) -> Net-(U13-Pad13)
- U13 pad 14: (no net) -> +5V
- U13 pad 2: /Control Logic/A15 -> /A15
- U13 pad 5: /Control Logic/CLK -> /CLK
- U13 pad 7: (no net) -> Earth
- U17 pad 10: Net-(U17-Pad10) -> /A12
- U17 pad 2: /Control Logic/A14 -> /A14
- U17 pad 4: /Control Logic/A14 -> /A14
- U17 pad 5: /Control Logic/A4 -> /A4
- U17 pad 6: Net-(U17-Pad10) -> Net-(U13-Pad13)
- U17 pad 8: Net-(U17-Pad8) -> /RAMOE
- U17 pad 9: /ROMCS -> /A13
- U4 pad 10: /CS2Via2 -> (no net)
- U4 pad 11: Net-(U17-Pad8) -> (no net)
- U4 pad 5: /HLT -> (no net)
- U4 pad 6: Net-(U4-Pad6) -> (no net)
- U5 pad 10: Net-(U4-Pad6) -> /HLT
- U5 pad 11: /RAMOE -> (no net)
- U5 pad 12: /Control Logic/A13 -> (no net)
- U5 pad 13: /Control Logic/A12 -> (no net)
Routing:
- net Earth: track 0.00 -> 1079.5 mm, vias 0 -> 1
- net +5V: track 0.00 -> 960.1 mm
- net /R/W: track 0.00 -> 360.2 mm, vias 0 -> 3
- net /CLK: track 0.00 -> 329.6 mm, vias 0 -> 1
- net /D0: track 0.00 -> 298.1 mm
- net /D6: track 0.00 -> 286.2 mm, vias 0 -> 2
- net /D4: track 0.00 -> 283.6 mm, vias 0 -> 1
- net /D1: track 0.00 -> 281.8 mm
- net /D2: track 0.00 -> 276.1 mm
- net /A1: track 0.00 -> 272.7 mm, vias 0 -> 1
- net /D5: track 0.00 -> 272.5 mm, vias 0 -> 1
- net /A0: track 0.00 -> 271.5 mm
- net /D7: track 0.00 -> 263.5 mm, vias 0 -> 1
- net /A12: track 0.00 -> 259.9 mm
- net /D3: track 0.00 -> 257.4 mm, vias 0 -> 1
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Other:
- board text added: "+"
- board text added: "Address Decoding"
- board text added: "BE6502 V2 Rev B"
- board text added: "Button"
- board text added: "Chip"
- board text added: "Clock Logic"
- board text added: "Reset Select"
- board text removed: "BE6502 V2 Rev A"
- board text removed: "Control Logic"
