File: clock.kicad_sch (KiCad schematic)
At the start: 39 parts, among them SW1 Step, SW12 RESET, SW2 Clk Source, SW2 Run / Step, U1 LM555, U15 LM555, U2 LM555, U3 LM555, U4 74LS04, U5 74LS08, U6 74LS32, X1 ACO-xxxMHz

Commit message: intermediate commit
Parts:
- added C10 (x5): 0.1µF, Capacitor_THT:C_Disc_D4.3mm_W1.9mm_P5.00mm, symbol Device:C
- added J1: Conn_01x03_Pin, Connector_PinSocket_1.27mm:PinSocket_1x03_P1.27mm_Vertical, symbol Connector:Conn_01x03_Pin
- added R10: 1k, Resistor_THT:R_Axial_DIN0207_L6.3mm_D2.5mm_P7.62mm_Horizontal, symbol Device:R
- added U4: 74LS04, Package_DIP:DIP-14_W7.62mm, symbol 8bit-computer-rescue:74LS04-8bit-computer-rescue
- renumbered C22 to C7, R22 to R12, R21 to R13, R23 to R14, SW12 to SW4, U15 to U7
Connections:
- net GND: now also U4.7 (GND); no longer C1.2, C10.2, C2.2, C2.2, C3.2, C4.2, C5.2, C6.2, C7.2, R13.2, R7.1, R7.1, R7.1, R7.2, SW1.1, SW2.2 (B), U1.1 (GND), U2.1 (GND), U3.1 (GND), U3.6 (THR), U7.1 (GND), X1.7 (GND)
- net HLT: now also R10.2
- net Reset: now also J1.2 (Pin_2); no longer R14.2, U7.7 (DIS)
- net VCC: now also U4.14 (VCC); no longer C1.1, C10.1, R1.1, R14.1, R3.1, R4.1, R5.1, R6.1, SW4.1, U1.4 (R), U1.8 (VCC), U2.4 (R), U2.8 (VCC), U3.8 (VCC), U7.4 (R), U7.8 (VCC)
- net at R12.2, R13.1, SW4.2: now also U4.9
- new net: J1.1 (Pin_1), R14.2, U7.7 (DIS)
- new net: J1.3 (Pin_3), U4.8
- new net +5V: C1.1, C10.1, C10.1, C10.1, C10.1, C10.1, C10.1, R1.1, R10.1, R14.1, R3.1, R4.1, R5.1, R6.1, SW4.1, U1.4 (R), U1.8 (VCC), U2.4 (R), U2.8 (VCC), U3.8 (VCC), U7.4 (R), U7.8 (VCC)
- new net Earth: C1.2, C10.2, C10.2, C10.2, C10.2, C10.2, C10.2, C2.2, C2.2, C3.2, C4.2, C5.2, C6.2, C7.2, R13.2, R7.1, R7.1, R7.1, R7.2, SW1.1, SW2.2 (B), U1.1 (GND), U2.1 (GND), U3.1 (GND), U3.6 (THR), U7.1 (GND), X1.7 (GND)
Other:
- moved on the sheet: C1, C10

Commit message: interm commit
Parts:
- added J11: Halt, Connector_Pin:Pin_D1.0mm_L10.0mm, symbol Connector:Conn_01x01_Pin
Connections:
- net HLT renamed Halt
- net Halt: now also J11.1 (Pin_1)

Commit message: An other interm relase
Parts:
- J11: value Halt -> HLT
Connections:
- net Halt renamed HLT
Changed lines of the file:
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@@
 		)
 	)
-	(hierarchical_label "Halt"
+	(hierarchical_label "HLT"
 		(shape input)
 		(at 42.545 150.495 270)
@@
 			)
 		)
-		(property "Value" "Halt"
+		(property "Value" "HLT"
 			(at 36.195 149.225 0)
 			(effects

Commit message: Fix Oops...
Parts:
- removed U4: 74LS04, Package_DIP:DIP-14_W7.62mm, symbol 8bit-computer-rescue:74LS04-8bit-computer-rescue
- J1: footprint Connector_PinSocket_1.27mm:PinSocket_1x03_P1.27mm_Vertical -> Connector_PinSocket_2.54mm:PinSocket_1x03_P2.54mm_Vertical
Connections:
- net HLT: now also U5.10
Changed lines of the file:
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@@
 	(wire
 		(pts
-			(xy 42.545 147.32) (xy 64.77 147.32)
+			(xy 42.545 147.32) (xy 160.02 147.32)
 		)
 		(stroke
@@
 	(wire
 		(pts
-			(xy 87.63 147.32) (xy 160.02 147.32)
-		)
-		(stroke
-			(width 0)
-			(type default)
-		)
-	)
-	(wire
-		(pts
 			(xy 39.37 77.47) (xy 50.8 77.47)
 		)
@@
 	(symbol
 		(lib_id "8bit-computer-rescue:74LS04-8bit-computer-rescue")
-		(at 76.2 147.32 0)
-		(unit 4)
-		(exclude_from_sim no)
-		(in_bom yes)
-		(on_board yes)
-		(dnp no)
-		(property "Reference" "U4"
-			(at 81.153 144.399 0)
-			(effects
-				(font
-					(size 1.27 1.27)
-				)
-			)
-		)
-		(property "Value" "74LS04"
-			(at 81.026 150.495 0)
-			(effects
-				(font
-					(size 1.27 1.27)
-				)
-			)
-		)
-		(property "Footprint" "Package_DIP:DIP-14_W7.62mm"
-			(at 76.2 147.32 0)
-			(effects
-				(font
-					(size 1.27 1.27)
-				)
-				(hide yes)
-			)
-		)
-		(property "Datasheet" ""
-			(at 76.2 147.32 0)
-			(effects
-				(font
-					(size 1.27 1.27)
-				)
-				(hide yes)
-			)
-		)
-		(property "Description" ""
-			(at 76.2 147.32 0)
-			(effects
-				(font
-					(size 1.27 1.27)
-				)
-				(hide yes)
-			)
-		)
-		(pin "14"
-		)
-		(pin "7"
-		)
-		(pin "1"
-		)
-		(pin "2"
-		)
-		(pin "3"
-		)
-		(pin "4"
-		)
-		(pin "5"
-		)
-		(pin "6"
-		)
-		(pin "8"
-		)
-		(pin "9"
-		)
-		(pin "10"
-		)
-		(pin "11"
-		)
-		(pin "12"
-		)
-		(pin "13"
-		)
-		(instances
-			(project "8bit-computer"
-				(path "/0e1a93c4-fdde-4b8f-a97d-016b71cdd04f/00000000-0000-0000-0000-00005b533ecb"
-					(reference "U4")
-					(unit 4)
-				)
-			)
-			(project "BenEater-6502"
-				(path "/64020bd5-bae0-49a1-9410-23726bcfaf48/5a49408d-bc6d-4641-a815-21b24906e7e4"
-					(reference "U4")
-					(unit 3)
-				)
-			)
-		)
-	)
-	(symbol
-		(lib_id "8bit-computer-rescue:74LS04-8bit-computer-rescue")
 		(at 223.52 107.95 0)
 		(unit 6)
@@
 			)
 		)
-		(property "Footprint" "Connector_PinSocket_1.27mm:PinSocket_1x03_P1.27mm_Vertical"
+		(property "Footprint" "Connector_PinSocket_2.54mm:PinSocket_1x03_P2.54mm_Vertical"
 			(at 110.49 180.975 0)
 			(effects

Commit message: updated plots
Changed lines of the file:
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@@
 			)
 		)
-		(property "Description" ""
+		(property "Description" "X1 / Generator"
 			(at 223.52 121.92 0)
 			(effects
@@
 					(size 1.27 1.27)
 				)
-				(hide yes)
 			)
 		)

Commit message: It works
Parts:
- R10: value 1k -> 10k
Changed lines of the file:
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@@
 			)
 		)
-		(property "Value" "1k"
+		(property "Value" "10k"
 			(at 42.545 135.89 90)
 			(effects
