File: expansion.kicad_sch (KiCad schematic)
At the start: 25 parts, among them J12 Conn_01x10, J13 Conn_01x10, J2 Conn_01x02, J3 Barrel Jack, J4 Logic Probe, J5 Conn_02x20_Counter_Clockwise, J6 Conn_02x20_Counter_Clockwise, SW2 Power, U14 W65C22NxP

Commit message: It works
Parts:
- added D8: SB140, Diode_THT:D_DO-41_SOD81_P10.16mm_Horizontal, symbol Diode:SB140
Connections:
- net IRQ: now also D8.2 (A); no longer U14.21 (~{IRQ})
- new net: D8.1 (K), U14.21 (~{IRQ})
Changed lines of the file:
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@@
 	(wire
 		(pts
-			(xy 34.798 70.612) (xy 41.91 70.612)
-		)
-		(stroke
-			(width 0)
-			(type default)
-		)
-	)
-	(wire
-		(pts
 			(xy 218.44 87.63) (xy 224.79 87.63)
 		)
@@
 	(wire
 		(pts
+			(xy 19.304 70.612) (xy 21.59 70.612)
+		)
+		(stroke
+			(width 0)
+			(type default)
+		)
+	)
+	(wire
+		(pts
 			(xy 85.09 78.232) (xy 85.09 82.55)
 		)
@@
 	(wire
 		(pts
+			(xy 29.21 70.612) (xy 41.91 70.612)
+		)
+		(stroke
+			(width 0)
+			(type default)
+		)
+	)
+	(wire
+		(pts
 			(xy 218.44 59.69) (xy 224.79 59.69)
 		)
@@
 	(hierarchical_label "IRQ"
 		(shape bidirectional)
-		(at 34.798 70.612 180)
+		(at 19.304 70.612 180)
 		(fields_autoplaced yes)
 		(effects
@@
 					(unit 1)
 				)
+			)
+		)
+	)
+	(symbol
+		(lib_id "Diode:SB140")
+		(at 25.4 70.612 180)
+		(unit 1)
+		(exclude_from_sim no)
+		(in_bom yes)
+		(on_board yes)
+		(dnp no)
+		(fields_autoplaced yes)
+		(property "Reference" "D8"
+			(at 25.7175 64.77 0)
+			(effects
+				(font
+					(size 1.27 1.27)
+				)
+			)
+		)
+		(property "Value" "SB140"
+			(at 25.7175 67.31 0)
+			(effects
+				(font
+					(size 1.27 1.27)
+				)
+			)
+		)
+		(property "Footprint" "Diode_THT:D_DO-41_SOD81_P10.16mm_Horizontal"
+			(at 25.4 66.167 0)
+			(effects
+				(font
+					(size 1.27 1.27)
+				)
+				(hide yes)
+			)
+		)
+		(property "Datasheet" "http://www.diodes.com/_files/datasheets/ds23022.pdf"
+			(at 25.4 70.612 0)
+			(effects
+				(font
+					(size 1.27 1.27)
+				)
+				(hide yes)
+			)
+		)
+		(property "Description" "40V 1A Schottky Barrier Rectifier Diode, DO-41"
+			(at 25.4 70.612 0)
+			(effects
+				(font
+					(size 1.27 1.27)
+				)
+				(hide yes)
+			)
+		)
+		(pin "2"
+		)
+		(pin "1"
+		)
+		(instances
+			(project "BenEater-6502"
+				(path "/64020bd5-bae0-49a1-9410-23726bcfaf48/16aa598a-cc79-4ffe-8299-2b52f0e64f5a"
+					(reference "D8")
+					(unit 1)
+				)
