File: serial.kicad_sch (KiCad schematic)
At the start: 16 parts, among them J1 Conn_01x09, J10 Conn_01x03_Pin, U13 W65C51NxP, U14 MAX232N, Y1 Crystal

Commit message: interm commit
Parts:
- renumbered C17 to C20, C17 to C21, C20 to C22, C18 to C23, C19 to C24, C17 to C25, C17 to C26, D5 to D8, J1 to J7, J1 to J8, J1 to J9, R13 to R24, U13 to U15, U14 to U16

Commit message: An other interm relase
Parts:
- J7, J8, J9: footprint Connector_PinSocket_1.27mm:PinSocket_1x09_P1.27mm_Vertical -> Connector_PinSocket_2.54mm:PinSocket_1x09_P2.54mm_Vertical
Changed lines of the file:
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@@
 			)
 		)
-		(property "Footprint" "Connector_PinSocket_1.27mm:PinSocket_1x09_P1.27mm_Vertical"
+		(property "Footprint" "Connector_PinSocket_2.54mm:PinSocket_1x09_P2.54mm_Vertical"
 			(at 200.025 66.04 0)
 			(effects
@@
 			)
 		)
-		(property "Footprint" "Connector_PinSocket_1.27mm:PinSocket_1x09_P1.27mm_Vertical"
+		(property "Footprint" "Connector_PinSocket_2.54mm:PinSocket_1x09_P2.54mm_Vertical"
 			(at 77.47 98.425 0)
 			(effects
@@
 			)
 		)
-		(property "Footprint" "Connector_PinSocket_1.27mm:PinSocket_1x09_P1.27mm_Vertical"
+		(property "Footprint" "Connector_PinSocket_2.54mm:PinSocket_1x09_P2.54mm_Vertical"
 			(at 217.17 66.04 0)
 			(effects

Commit message: Fix Oops...
Parts:
- C25, C26: value .1uf -> 0.1uf
- J10: footprint Connector_PinSocket_1.27mm:PinSocket_1x03_P1.27mm_Vertical -> Connector_PinSocket_2.54mm:PinSocket_1x03_P2.54mm_Vertical
Changed lines of the file:
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@@
 			)
 		)
-		(property "Value" ".1uf"
+		(property "Value" "0.1uf"
 			(at 85.725 158.115 0)
 			(effects
@@
 			)
 		)
-		(property "Footprint" "Connector_PinSocket_1.27mm:PinSocket_1x03_P1.27mm_Vertical"
+		(property "Footprint" "Connector_PinSocket_2.54mm:PinSocket_1x03_P2.54mm_Vertical"
 			(at 102.87 122.555 0)
 			(effects
@@
 			)
 		)
-		(property "Value" ".1uf"
+		(property "Value" "0.1uf"
 			(at 74.295 158.115 0)
 			(effects

Commit message: Closer yet
Parts:
- removed D8: SB140, Diode_THT:D_DO-41_SOD81_P10.16mm_Horizontal, symbol Diode:SB140
Connections:
- net IRQ: now also U15.26 (~{IRQ})
Changed lines of the file:
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@@
-	(wire
-		(pts
-			(xy 38.735 61.595) (xy 41.275 61.595)
-		)
-		(stroke
-			(width 0)
-			(type default)
-		)
-	)
 	(wire
 		(pts
@@
 	(wire
 		(pts
-			(xy 27.305 61.595) (xy 31.115 61.595)
+			(xy 27.305 61.595) (xy 41.275 61.595)
 		)
 		(stroke
@@
 					(unit 1)
 				)
-			)
-		)
-	)
-	(symbol
-		(lib_id "Diode:SB140")
-		(at 34.925 61.595 180)
-		(unit 1)
-		(exclude_from_sim no)
-		(in_bom yes)
-		(on_board yes)
-		(dnp no)
-		(property "Reference" "D8"
-			(at 32.385 60.325 0)
-			(effects
-				(font
-					(size 1.27 1.27)
-				)
-			)
-		)
-		(property "Value" "SB140"
-			(at 35.2425 57.785 0)
-			(effects
-				(font
-					(size 1.27 1.27)
-				)
-				(hide yes)
-			)
-		)
-		(property "Footprint" "Diode_THT:D_DO-41_SOD81_P10.16mm_Horizontal"
-			(at 34.925 57.15 0)
-			(effects
-				(font
-					(size 1.27 1.27)
-				)
-				(hide yes)
-			)
-		)
-		(property "Datasheet" "http://www.diodes.com/_files/datasheets/ds23022.pdf"
-			(at 34.925 61.595 0)
-			(effects
-				(font
-					(size 1.27 1.27)
-				)
-				(hide yes)
-			)
-		)
-		(property "Description" ""
-			(at 34.925 61.595 0)
-			(effects
-				(font
-					(size 1.27 1.27)
-				)
-				(hide yes)
-			)
-		)
-		(pin "1"
-		)
-		(pin "2"
-		)
-		(instances
-			(project "BenEater-6502"
-				(path "/64020bd5-bae0-49a1-9410-23726bcfaf48/5be250a5-29bf-4920-8282-0800b279cae0"
-					(reference "D8")
-					(unit 1)
-				)

Commit message: Fixed the addressing Still not fixed
Parts:
- J10: value Conn_01x03_Pin -> RTS Select
Connections:
- net A12 renamed CS1Serial

Commit message: It works
Parts:
- added D7: SB140, Diode_THT:D_DO-41_SOD81_P10.16mm_Horizontal, symbol Diode:SB140
Connections:
- net IRQ: now also D7.2 (A); no longer U15.26 (~{IRQ})
- new net: D7.1 (K), U15.26 (~{IRQ})
